File: bottom-module.kicad_pcb (KiCad board)
At the start: 2 copper layers, 135.6 x 83.3 mm, 15 parts, among them J10 Conn_02x12_Odd_Even, J13 PROTO1, J18 PROTO1, J5 Screw_Terminal_01x06, J6 Conn_02x12_Odd_Even, J8 Screw_Terminal_01x02, J9 Conn_02x12_Odd_Even

Commit message: Clean module
Signed-off-by: Martin Ribelotta <martinribelotta@gmail.com>
Parts:
- removed J10, J6, J9: Conn_02x12_Odd_Even, Connector_PinSocket_2.54mm:PinSocket_2x12_P2.54mm_Vertical
- removed J13, J18: PROTO1, Connector_PinHeader_2.54mm:PinHeader_2x10_P2.54mm_Vertical
- removed J5: Screw_Terminal_01x06, Connectors_Phoenix:PhoenixContact_MC-G_06x5.08mm_Angled
- removed J8: Screw_Terminal_01x02, Connectors_Phoenix:PhoenixContact_MC-G_02x5.08mm_Angled
